File: Kicad/RAF.sch (KiCad schematic (older format))
At the start: 29 parts, among them J1 CONN_01X03, J2 CONN_01X03, J3 SOL, J4 CONN_01X03, J5 PUMP, J6 WS2811-OUT, J7 I2C, P1 Power, P2 Analog, P3 Digital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

Commit message: layout and gerbers
Parts:
- added OSHW1: OSHW, RAF_Libs:OSHW_6mm, symbol OSHW
- added WYO1: LOGO_WL, RAF_Libs:logo_wyo_butterfly_small, symbol LOGO_WL
Changed lines of the file:
@@
 	3600 4650 3600 4750
 Connection ~ 3600 4650
+$Comp
+L OSHW OSHW1
+U 1 1 5981F4A6
+P 5950 4550
+F 0 "OSHW1" H 5950 4500 40  0001 C CNN
+F 1 "OSHW" H 5950 4650 40  0001 C CNN
+F 2 "RAF_Libs:OSHW_6mm" H 5950 4550 60  0001 C CNN
+F 3 "" H 5950 4550 60  0000 C CNN
+	1    5950 4550
+	1    0    0    -1
+$EndComp
+$Comp
+L LOGO_WL WYO1
+U 1 1 5981F4F6
+P 10100 7000
+F 0 "WYO1" H 10100 6864 60  0001 C CNN
+F 1 "LOGO_WL" H 10100 7136 60  0001 C CNN
+F 2 "RAF_Libs:logo_wyo_butterfly_small" H 10100 7000 60  0001 C CNN
+F 3 "" H 10100 7000 60  0001 C CNN
+	1    10100 7000
+	1    0    0    -1
+$EndComp
 $EndSCHEMATC
