File: Kicad/RAF.kicad_pcb (KiCad board)
At the start: 2 copper layers, 68.6 x 53.3 mm, 8 parts, among them P1 Power, P2 Analog, P3 Digital, P4 Digital, P5 CONN_01X01, P6 CONN_01X01, P7 CONN_01X01, P8 CONN_01X01

Commit message: new parts, initial layout, backup of switcher design
Parts:
- removed P5, P6, P7, P8: CONN_01X01, Socket_Arduino_Uno:Arduino_1pin
- added C1: .1uF, Capacitors_SMD:C_0805_HandSoldering, F.Cu at (154.8, 115.1)
- added C2: 2.2uF, Capacitors_SMD:CP_Elec_4x5.7, F.Cu at (163.1, 98.4)
- added J1: CONN_01X03, Pin_Headers:Pin_Header_Straight_1x03_Pitch2.54mm, F.Cu at (164.3, 80.6)
- added J2: CONN_01X03, Pin_Headers:Pin_Header_Straight_1x03_Pitch2.54mm, F.Cu at (161.8, 80.6)
- added J3: SOL, Terminal_Blocks:TerminalBlock_Pheonix_PT-3.5mm_2pol, F.Cu at (173.9, 117.1)
- added J4: CONN_01X03, Pin_Headers:Pin_Header_Straight_1x03_Pitch2.54mm, F.Cu at (159.3, 80.6)
- added J5: PUMP, Terminal_Blocks:TerminalBlock_Pheonix_PT-3.5mm_2pol, F.Cu at (173.9, 108.8)
- added J6: WS2811-OUT, Pin_Headers:Pin_Header_Straight_1x03_Pitch2.54mm, F.Cu at (123.7, 83.2)
- added J7: I2C, Pin_Headers:Pin_Header_Straight_1x04_Pitch2.54mm, F.Cu at (115.1, 75.5)
- added JOY1: AnalogJoystick, RAF_Libs:Adafruit-thumb-joystick, F.Cu at (121.2, 101.0)
- added JP1: Jumper_NC_Small, RAF_Libs:0805_jumper, F.Cu at (131.0, 117.4)
- added JP2: Jumper_NC_Small, RAF_Libs:0805_jumper, F.Cu at (131.0, 119.4)
- added JP3: Jumper_NC_Small, RAF_Libs:0805_jumper, F.Cu at (131.0, 121.4)
- added JP4: Jumper_NC_Small, RAF_Libs:0805_jumper, F.Cu at (131.0, 123.4)
- added LDR1: LDR03, RAF_Libs:Resistor_LDR_4.9x4.2_RM2.54, F.Cu at (152.0, 82.2)
- added Q1: FDC6305N, TO_SOT_Packages_SMD:SuperSOT-6, F.Cu at (175.8, 98.4)
- added R1: 22K, Resistors_SMD:R_0805_HandSoldering, F.Cu at (143.4, 87.5)
- added R2: 10K, Resistors_SMD:R_0805_HandSoldering, F.Cu at (170.7, 85.7)
- added R5: 100K, Resistors_SMD:R_0805_HandSoldering, F.Cu at (169.4, 94.6)
- added R6: 100K, Resistors_SMD:R_0805_HandSoldering, F.Cu at (169.4, 99.7)
- added R7: 100K, Resistors_SMD:R_0805_HandSoldering, F.Cu at (175.8, 92.1)
- added S1: SPST-M, Buttons_Switches_SMD:SW_SPST_PTS645, F.Cu at (140.0, 101.4)
- added TH1: Thermistor, Resistors_SMD:R_0805_HandSoldering, F.Cu at (170.7, 81.9)
- added U1: RGB_WS2811B, LEDs:LED_WS2812B-PLCC4, F.Cu at (130.6, 83.1)
- added U2: LF60CDT, RAF_Libs:DPak, B.Cu at (155.5, 99.0)
Connections:
- P2 pad 5: /A4(SDA) -> /A4
- P2 pad 6: /A5(SCL) -> /A5
Routing:
- net +5V: track 0.00 -> 65.3 mm
- net /Vin: track 0.00 -> 36.3 mm, vias 0 -> 1
- net GND: track 0.00 -> 31.0 mm, vias 0 -> 1
- net /2: track 0.00 -> 20.7 mm
- net /A2: track 0.00 -> 16.1 mm
- net /3(**): track 0.00 -> 6.13 mm
- net /6(**): track 0.00 -> 5.08 mm
- net /5(**): track 0.00 -> 5.08 mm
- net /A3: track 0.00 -> 3.81 mm
- added copper zone on B.Cu, net GND

Commit message: layout and gerbers
Parts:
- added OSHW1: OSHW, RAF_Libs:OSHW_6mm, F.Cu at (136.7, 89.5)
- added WYO1: LOGO_WL, RAF_Libs:logo_wyo_butterfly_small, B.Cu at (125.7, 123.6)
- JP1, JP2, JP3, JP4: moved to B.Cu
- moved JP4 17.1 mm to (141.2, 109.6)
- moved JP3 14.1 mm to (141.2, 111.6)
- moved JP2 11.7 mm to (141.2, 113.6)
- moved JP1 10.3 mm to (141.2, 115.6)
- moved C1 9.39 mm to (162.8, 110.1)
- moved S1 3.01 mm to (143.0, 101.2)
- moved J7 0.28 mm to (114.8, 75.6)
Routing:
- net +5V: track 65.3 -> 157.2 mm
- net /A3: track 3.81 -> 94.2 mm, vias 0 -> 1
- net GND: track 31.0 -> 98.4 mm, vias 1 -> 2
- net /A2: track 16.1 -> 82.9 mm, vias 0 -> 1
- net /SVCC: track 0.00 -> 54.3 mm, vias 0 -> 2
- net /A1: track 0.00 -> 49.9 mm
- net /A0: track 0.00 -> 49.3 mm
- net /12(MISO): track 0.00 -> 33.1 mm, vias 0 -> 1
- net /9(**): track 0.00 -> 30.2 mm, vias 0 -> 1
- net /Vin: track 36.3 -> 58.5 mm
- net /8: track 0.00 -> 22.1 mm
- net Net-(J3-Pad2): track 0.00 -> 19.3 mm
- net /A4(SDA): track 0.00 -> 15.2 mm
- net /A5(SCL): track 0.00 -> 13.5 mm
- net Net-(Q1-Pad3): track 0.00 -> 8.91 mm
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Other:
- net class .5 added: clearance 0.2, trace_width 0.5, via_dia 0.6, via_drill 0.4
- net class .75 added: clearance 0.2, trace_width 0.75, via_dia 0.6, via_drill 0.4
- board text added: "+5V"
- board text added: "3"
- board text added: "5"
- board text added: "6"
- board text added: "A0"
- board text added: "A1"
- board text added: "A2"
- board text added: "A3"
- board text added: "B"
- board text added: "DO"
- board text added: "GND"
- board text added: "Light"
- board text added: "R"
- board text added: "Ready Aim Fire V2.0"
- board text added: "SCL"
- board text added: "SDA"
- board text added: "Temp"
- board text added: "W"
- board text added: "Wyolum.com"
- board text added: "X"
- board text added: "Y"
- board text removed: "1"

Commit message: add pin 1 indications for LED and mosfet
Other:
- board text added: "1"
Changed lines of the file:
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@@
     (links 74)
     (no_connects 14)
-    (area 104.572999 72.949999 180.9634 126.6402)
+    (area 94.515267 65.752135 180.9634 126.728827)
     (thickness 1.6)
-    (drawings 52)
+    (drawings 54)
     (tracks 188)
     (zones 0)
@@
       (xy 1.953951 0.762056) (xy 1.996221 0.771764) (xy 2.048145 0.753984)) (layer B.SilkS) (width 0.01))
   )
+  (gr_text 1 (at 126.492 80.137) (layer F.SilkS)
+    (effects (font (size 0.8 0.8) (thickness 0.15)))
+  )
+  (gr_text 1 (at 173.228 96.647) (layer F.SilkS)
+    (effects (font (size 0.8 0.8) (thickness 0.15)))
+  )
   (dimension 53.596408 (width 0.3) (layer Dwgs.User)

Commit message: add labels for the mosfet terminals
Other:
- board text added: "6V"
- board text added: "Vin"
Changed lines of the file:
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@@
     (area 94.515267 65.752135 180.9634 126.728827)
     (thickness 1.6)
-    (drawings 54)
+    (drawings 56)
     (tracks 188)
     (zones 0)
@@
     (visible_elements FFFEFF7F)
     (pcbplotparams
-      (layerselection 0x00030_80000001)
+      (layerselection 0x01000_00000000)
       (usegerberextensions false)
       (excludeedgelayer true)
@@
       (padsonsilk false)
       (subtractmaskfromsilk false)
-      (outputformat 1)
+      (outputformat 5)
       (mirror false)
-      (drillshape 1)
+      (drillshape 0)
       (scaleselection 1)
-      (outputdirectory ""))
+      (outputdirectory RAF_pdf/))
   )
   (net 0 "")
@@
     (add_net GND)
   )
+  (module LEDs:LED_WS2812B-PLCC4 (layer F.Cu)
+    (at 130.6449 83.1469)
+    (descr http://www.world-semi.com/uploads/soft/150522/1-150522091P5.pdf)
+    (tags "LED NeoPixel")
+    (attr smd)
+    (fp_text reference U1 (at 0 -3.5) (layer F.SilkS)
+      (effects (font (size 1 1) (thickness 0.15)))
+    )
+    (fp_text value RGB_WS2811B (at 0 4) (layer F.Fab)
+      (effects (font (size 1 1) (thickness 0.15)))
+    )
+    (fp_line (start 3.75 -2.85) (end -3.75 -2.85) (layer F.CrtYd) (width 0.05))
+    (fp_line (start 3.75 2.85) (end 3.75 -2.85) (layer F.CrtYd) (width 0.05))
+    (fp_line (start -3.75 2.85) (end 3.75 2.85) (layer F.CrtYd) (width 0.05))
+    (fp_line (start -3.75 -2.85) (end -3.75 2.85) (layer F.CrtYd) (width 0.05))
+    (fp_line (start 2.5 1.5) (end 1.5 2.5) (layer F.SilkS) (width 0.1))
+    (fp_line (start -2.5 -2.5) (end -2.5 2.5) (layer F.SilkS) (width 0.1))
+    (fp_line (start -2.5 2.5) (end 2.5 2.5) (layer F.SilkS) (width 0.1))
+    (fp_line (start 2.5 2.5) (end 2.5 -2.5) (layer F.SilkS) (width 0.1))
+    (fp_line (start 2.5 -2.5) (end -2.5 -2.5) (layer F.SilkS) (width 0.1))
+    (fp_circle (center 0 0) (end 0 -2) (layer F.SilkS) (width 0.1))
+    (pad 3 smd rect (at 2.5 1.6) (size 1.6 1) (layers F.Cu F.Paste F.Mask)
+      (net 4 GND))
+    (pad 4 smd rect (at 2.5 -1.6) (size 1.6 1) (layers F.Cu F.Paste F.Mask)
+      (net 14 /8))
+    (pad 2 smd rect (at -2.5 1.6) (size 1.6 1) (layers F.Cu F.Paste F.Mask)
+      (net 32 /LED_OUT))
+    (pad 1 smd rect (at -2.5 -1.6) (size 1.6 1) (layers F.Cu F.Paste F.Mask)
+      (net 3 +5V))
+    (model ${KISYS3DMOD}/LEDs.3dshapes/LED_WS2812B-PLCC4.wrl
+      (at (xyz 0 0 0))
+      (scale (xyz 0.39 0.39 0.39))
+      (rotate (xyz 0 0 180))
+    )
+  )
   (module Socket_Arduino_Uno:Socket_Strip_Arduino_1x08 locked (layer F.Cu)
     (at 138.938 123.825)
@@
       (net 4 GND))
     (model ${KISYS3DMOD}/Pin_Headers.3dshapes/Pin_Header_Straight_1x03_Pitch2.54mm.wrl
-      (at (xyz 0 0 0))
-      (scale (xyz 1 1 1))
-      (rotate (xyz 0 0 0))
+      (at (xyz 0 -0.1 0))
+      (scale (xyz 1 1 1))
+      (rotate (xyz 0 0 90))
     )
   )
@@
       (net 4 GND))
     (model ${KISYS3DMOD}/Pin_Headers.3dshapes/Pin_Header_Straight_1x03_Pitch2.54mm.wrl
-      (at (xyz 0 0 0))
-      (scale (xyz 1 1 1))
-      (rotate (xyz 0 0 0))
+      (at (xyz 0 -0.1 0))
+      (scale (xyz 1 1 1))
+      (rotate (xyz 0 0 90))
     )
   )
@@
       (net 4 GND))
     (model ${KISYS3DMOD}/Pin_Headers.3dshapes/Pin_Header_Straight_1x03_Pitch2.54mm.wrl
-      (at (xyz 0 0 0))
-      (scale (xyz 1 1 1))
-      (rotate (xyz 0 0 0))
+      (at (xyz 0 -0.1 0))
+      (scale (xyz 1 1 1))
+      (rotate (xyz 0 0 90))
     )
   )
@@
       (net 4 GND))
     (model ${KISYS3DMOD}/Pin_Headers.3dshapes/Pin_Header_Straight_1x03_Pitch2.54mm.wrl
-      (at (xyz 0 0 0))
-      (scale (xyz 1 1 1))
-      (rotate (xyz 0 0 0))
+      (at (xyz 0 -0.1 0))
+      (scale (xyz 1 1 1))
+      (rotate (xyz 0 0 90))
     )
   )
@@
       (net 4 GND))
     (model ${KISYS3DMOD}/Pin_Headers.3dshapes/Pin_Header_Straight_1x04_Pitch2.54mm.wrl
-      (at (xyz 0 0 0))
-      (scale (xyz 1 1 1))
-      (rotate (xyz 0 0 0))
+      (at (xyz 0 -0.2 0))
+      (scale (xyz 1 1 1))
+      (rotate (xyz 0 0 90))
     )
   )
@@
       (scale (xyz 1 1 1))
       (rotate (xyz 0 0 0))
-    )
-  )
-  (module LEDs:LED_WS2812B-PLCC4 (layer F.Cu)
-    (at 130.6449 83.1469)
-    (descr http://www.world-semi.com/uploads/soft/150522/1-150522091P5.pdf)
-    (tags "LED NeoPixel")
-    (attr smd)
-    (fp_text reference U1 (at 0 -3.5) (layer F.SilkS)
-      (effects (font (size 1 1) (thickness 0.15)))
-    )
-    (fp_text value RGB_WS2811B (at 0 4) (layer F.Fab)
-      (effects (font (size 1 1) (thickness 0.15)))
-    )
-    (fp_line (start 3.75 -2.85) (end -3.75 -2.85) (layer F.CrtYd) (width 0.05))
-    (fp_line (start 3.75 2.85) (end 3.75 -2.85) (layer F.CrtYd) (width 0.05))
-    (fp_line (start -3.75 2.85) (end 3.75 2.85) (layer F.CrtYd) (width 0.05))
-    (fp_line (start -3.75 -2.85) (end -3.75 2.85) (layer F.CrtYd) (width 0.05))
-    (fp_line (start 2.5 1.5) (end 1.5 2.5) (layer F.Fab) (width 0.1))
-    (fp_line (start -2.5 -2.5) (end -2.5 2.5) (layer F.Fab) (width 0.1))
-    (fp_line (start -2.5 2.5) (end 2.5 2.5) (layer F.Fab) (width 0.1))
-    (fp_line (start 2.5 2.5) (end 2.5 -2.5) (layer F.Fab) (width 0.1))
-    (fp_line (start 2.5 -2.5) (end -2.5 -2.5) (layer F.Fab) (width 0.1))
-    (fp_line (start -3.5 -2.6) (end 3.5 -2.6) (layer F.SilkS) (width 0.12))
-    (fp_line (start -3.5 2.6) (end 3.5 2.6) (layer F.SilkS) (width 0.12))
-    (fp_line (start 3.5 2.6) (end 3.5 1.6) (layer F.SilkS) (width 0.12))
-    (fp_circle (center 0 0) (end 0 -2) (layer F.Fab) (width 0.1))
-    (pad 3 smd rect (at 2.5 1.6) (size 1.6 1) (layers F.Cu F.Paste F.Mask)
-      (net 4 GND))
-    (pad 4 smd rect (at 2.5 -1.6) (size 1.6 1) (layers F.Cu F.Paste F.Mask)
-      (net 14 /8))
-    (pad 2 smd rect (at -2.5 1.6) (size 1.6 1) (layers F.Cu F.Paste F.Mask)
-      (net 32 /LED_OUT))
-    (pad 1 smd rect (at -2.5 -1.6) (size 1.6 1) (layers F.Cu F.Paste F.Mask)
-      (net 3 +5V))
-    (model ${KISYS3DMOD}/LEDs.3dshapes/LED_WS2812B-PLCC4.wrl
-      (at (xyz 0 0 0))
-      (scale (xyz 0.39 0.39 0.39))
-      (rotate (xyz 0 0 180))
     )
   )
@@
       (xy 1.953951 0.762056) (xy 1.996221 0.771764) (xy 2.048145 0.753984)) (layer B.SilkS) (width 0.01))
   )
+  (gr_text 6V (at 167.64 107.061 90) (layer F.SilkS)
+    (effects (font (size 1.5 1.5) (thickness 0.3)))
+  )
+  (gr_text Vin (at 167.64 115.697 90) (layer F.SilkS)
+    (effects (font (size 1.5 1.5) (thickness 0.3)))
+  )
   (gr_text 1 (at 126.492 80.137) (layer F.SilkS)
