File: kicad_v2/RAF.kicad_pcb (KiCad board)
At the start: 2 copper layers, 68.6 x 53.3 mm, 31 parts, among them J1 SERVO, J2 SERVO, J3 SOL, J4 SERVO, J5 PUMP, J6 WS2811-OUT, J7 I2C, P1 Power, P2 Analog, P3 Digital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

Commit message: RAF v3 Kicad WIP
Parts:
- added C3: 0.1uF, RAF_Libs:C_0805_HandSoldering, F.Cu at (121.2, 114.9)
- added C4: 0.1uF, RAF_Libs:C_0805_HandSoldering, F.Cu at (135.1, 101.0)
- added C5: 0.1uF, RAF_Libs:C_0805_HandSoldering, F.Cu at (141.5, 84.5)
- added C6: 0.1uF, RAF_Libs:C_0805_HandSoldering, F.Cu at (155.4, 84.5)
- added C7: 2.2uF, RAF_Libs:CP_Elec_4x5.7, F.Cu at (151.6, 84.5)
- added C8: 0.1uF, RAF_Libs:C_0805_HandSoldering, F.Cu at (121.2, 84.5)
- added C9: 0.1uF, RAF_Libs:C_0805_HandSoldering, F.Cu at (114.8, 84.5)
- added D1: SD3220, RAF_Libs:SMA_Handsoldering, F.Cu at (158.0, 116.2)
- added D2: SD3220, RAF_Libs:SMA_Handsoldering, F.Cu at (158.0, 106.0)
- C1: footprint Capacitors_SMD:C_0805_HandSoldering -> RAF_Libs:C_0805_HandSoldering
- C2: footprint Capacitors_SMD:CP_Elec_4x5.7 -> RAF_Libs:CP_Elec_4x5.7
- J1, J2, J4, J6: footprint Pin_Headers:Pin_Header_Straight_1x03_Pitch2.54mm -> RAF_Libs:Pin_Header_Straight_1x03_Pitch2.54mm
- J7: footprint Pin_Headers:Pin_Header_Straight_1x04_Pitch2.54mm -> RAF_Libs:Pin_Header_Straight_1x04_Pitch2.54mm
- P1, P4: footprint Socket_Arduino_Uno:Socket_Strip_Arduino_1x08 -> RAF_Libs:Socket_Strip_Arduino_1x08
- P2: footprint Socket_Arduino_Uno:Socket_Strip_Arduino_1x06 -> RAF_Libs:Socket_Strip_Arduino_1x06
- P3: footprint Socket_Arduino_Uno:Socket_Strip_Arduino_1x10 -> RAF_Libs:Socket_Strip_Arduino_1x10
- Q1: footprint TO_SOT_Packages_SMD:SuperSOT-6 -> RAF_Libs:SuperSOT-6
- R1, R2, R5, R6, R7, TH1: footprint Resistors_SMD:R_0805_HandSoldering -> RAF_Libs:R_0805_HandSoldering
- S1: footprint Buttons_Switches_SMD:SW_SPST_PTS645 -> RAF_Libs:SW_SPST_PTS645
- U1: footprint LEDs:LED_WS2812B-PLCC4 -> RAF_Libs:LED_WS2812B-PLCC4
- moved R2 66.2 mm to (114.8, 121.3), turned to 90 degrees
- moved TH1 64.3 mm to (119.9, 121.3), turned to 90 degrees
- moved OSHW1 50.6 mm to (142.7, 108.6)
- moved LDR1 43.9 mm to (132.6, 122.6), turned to 90 degrees
- moved WYO1 38.7 mm to (125.0, 121.3)
- moved R1 34.4 mm to (125.0, 121.3)
- moved U1 5.17 mm to (135.1, 85.7), turned to 270 degrees
- moved C2 4.44 mm to (158.0, 94.6)
- moved J6 3.18 mm to (126.9, 83.2)
- moved C1 2.01 mm to (151.6, 94.6)
- moved J3 0.64 mm to (165.6, 116.2)
- moved J5 0.61 mm to (165.6, 106.0)
- moved S1 0.36 mm to (142.7, 101.0)
Routing:
- removed copper zone on B.Cu, net GND
Other:
- board text added: "Ready Aim Fire V3.0"
- board text removed: "Ready Aim Fire V2.0"
