File: kicad_v2/RAF.sch (KiCad schematic (older format))
At the start: 31 parts, among them J1 SERVO, J2 SERVO, J3 SOL, J4 SERVO, J5 PUMP, J6 WS2811-OUT, J7 I2C, P1 Power, P2 Analog, P3 Digital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

Commit message: RAF v3 Kicad WIP
Parts:
- added C3, C4, C5, C6, C8, C9: 0.1uF, RAF_Libs:C_0805_HandSoldering, symbol C
- added C7: 2.2uF, RAF_Libs:CP_Elec_4x5.7, symbol CP
- added D1, D2: SD3220, RAF_Libs:SMA_Handsoldering, symbol D_Small
- C1: footprint Capacitors_SMD:C_0805_HandSoldering -> RAF_Libs:C_0805_HandSoldering
- C2: footprint Capacitors_SMD:CP_Elec_4x5.7 -> RAF_Libs:CP_Elec_4x5.7
- J1, J2, J4, J6: footprint Pin_Headers:Pin_Header_Straight_1x03_Pitch2.54mm -> RAF_Libs:Pin_Header_Straight_1x03_Pitch2.54mm
- J3, J5: footprint Terminal_Blocks:TerminalBlock_Pheonix_PT-3.5mm_2pol -> RAF_Libs:TerminalBlock_Pheonix_PT-5.0mm_2pol
- J7: footprint Pin_Headers:Pin_Header_Straight_1x04_Pitch2.54mm -> RAF_Libs:Pin_Header_Straight_1x04_Pitch2.54mm
- P1, P4: footprint Socket_Arduino_Uno:Socket_Strip_Arduino_1x08 -> RAF_Libs:Socket_Strip_Arduino_1x08
- P2: footprint Socket_Arduino_Uno:Socket_Strip_Arduino_1x06 -> RAF_Libs:Socket_Strip_Arduino_1x06
- P3: footprint Socket_Arduino_Uno:Socket_Strip_Arduino_1x10 -> RAF_Libs:Socket_Strip_Arduino_1x10
- Q1: footprint TO_SOT_Packages_SMD:SuperSOT-6 -> RAF_Libs:SuperSOT-6
- R1, R2, R5, R6, R7, TH1: footprint Resistors_SMD:R_0805_HandSoldering -> RAF_Libs:R_0805_HandSoldering
- S1: footprint Buttons_Switches_SMD:SW_SPST_PTS645 -> RAF_Libs:SW_SPST_PTS645
- U1: footprint LEDs:LED_WS2812B-PLCC4 -> RAF_Libs:LED_WS2812B-PLCC4
Connections:
- net +5V: now also C5.1, C8.1, C9.1
- net A0: now also C3.1
- net A1: now also C4.1
- net GND: now also C3.2, C4.2, C5.2, C6.2, C7.2, C8.2, C9.2
- net SVCC: now also C6.1, C7.1, D2.1 (K)
- net Vin: now also D1.1 (K)
- net at J3.2 (P2), Q1.6 (D): now also D1.2 (A)
- net at J5.2 (P2), Q1.4 (D): now also D2.2 (A)
Other:
- moved on the sheet: J3, J5, JOY1, JP1, JP2, JP3, JP4, Q1A, Q1B, R5, R6, R7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
