File: kicad_v2.1/RAF_adaJS.kicad_pcb (KiCad board)
At the start: 2 copper layers, 68.6 x 53.3 mm, 44 parts, among them J1 SERVO, J2 SERVO, J3 SOL, J4 SERVO, J5 PUMP, J6 WS2811-OUT, J7 I2C, P1 Power, P2 Analog, P3 Digital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

Commit message: seeed joystick revision
Parts:
- added S1: FIRE, RAF_Libs:SW_SPST_PTS645, F.Cu at (142.7, 101.0)
- JOY1: value SeeedJoystick -> AnalogJoystick; footprint RAF_Libs:SEEED-Joystick_v2 -> RAF_Libs:Adafruit-thumb-joystick
- moved WYO1 19.1 mm to (126.9, 115.6)
- moved OSHW1 10.9 mm to (142.7, 108.6)
- moved C3 8.91 mm to (121.2, 114.9), turned to 180 degrees
- moved JOY1 7.73 mm to (121.2, 101.0), turned to 0 degrees
- moved C4 7.62 mm to (135.1, 101.0), turned to 90 degrees
- moved JP3 5.71 mm to (137.7, 111.8)
- moved JP4 5.71 mm to (137.7, 109.9)
- moved JP2 1.91 mm to (137.7, 113.7)
- moved JP1 1.90 mm to (137.7, 115.6)
Routing:
- net GND: track 379.9 -> 356.4 mm, vias 9 -> 13
- net /A2: track 55.7 -> 70.1 mm
- net /A3: track 64.0 -> 77.4 mm
- net /12(MISO): track 50.9 -> 45.4 mm
- net /A1: track 58.2 -> 61.9 mm, vias 2 -> 1
- net +5V: track 160.2 -> 157.1 mm
- net /A0: track 50.4 -> 49.6 mm, vias 2 -> 1
- net /A4(SDA): track 18.9 -> 19.6 mm
