File: kicad_v2.1/RAF.kicad_pcb (KiCad board)
At the start: 2 copper layers, 68.6 x 53.3 mm, 45 parts, among them J1 SERVO, J2 SERVO, J3 SOL, J4 SERVO, J5 PUMP, J6 WS2811-OUT, J7 I2C, J8 AUX_TEST, P1 Power, P2 Analog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

Commit message: updated aux_test PCB
Routing:
- net +5V: track 171.8 -> 181.0 mm
- net GND: track 275.0 -> 280.2 mm
- net /Vin: track 80.4 -> 77.2 mm
- net /SVCC: track 106.5 -> 105.4 mm
Other:
- board text added: "SVCC"
- board text added: "Vin"

Commit message: edited values of C2,C7
Parts:
- C2, C7: value 2.2uF -> 22uF
Changed lines of the file:
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@@
       (effects (font (size 1 1) (thickness 0.15)))
     )
-    (fp_text value 2.2uF (at 0 -3.54 270) (layer F.Fab)
+    (fp_text value 22uF (at 0 -3.54 270) (layer F.Fab)
       (effects (font (size 1 1) (thickness 0.15)))
     )
@@
       (effects (font (size 1 1) (thickness 0.15)))
     )
-    (fp_text value 2.2uF (at 0 -3.54 270) (layer F.Fab)
-      (effects (font (size 1 1) (thickness 0.15)))
-    )
+    (fp_text value 22uF (at 0 -3.54 270) (layer F.Fab)
+      (effects (font (size 1 1) (thickness 0.15)))
+    )
